File: detector_block/detector_block.kicad_pcb (KiCad board)
At the start: 2 copper layers, 8.1 x 7.6 mm, 3 parts

Commit message: detector block
Other:
- board size 8.1 x 7.6 mm -> 8.9 x 8.9 mm
Changed lines of the file:
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@@
     (visible_elements 7FFEFF7F)
     (pcbplotparams
-      (layerselection 0x020f0_80000001)
+      (layerselection 0x010f0_80000001)
       (usegerberextensions true)
       (excludeedgelayer true)
@@
     )
   )
-  (gr_line (start 153.035 91.059) (end 144.907 91.059) (angle 90) (layer Edge.Cuts) (width 0.1))
-  (gr_line (start 144.907 91.059) (end 145.034 91.059) (angle 90) (layer Edge.Cuts) (width 0.1))
-  (gr_line (start 144.907 98.679) (end 144.907 91.059) (angle 90) (layer Edge.Cuts) (width 0.1))
-  (gr_line (start 153.035 98.679) (end 144.907 98.679) (angle 90) (layer Edge.Cuts) (width 0.1))
-  (gr_line (start 153.035 91.059) (end 153.035 98.679) (angle 90) (layer Edge.Cuts) (width 0.1))
+  (gr_line (start 144.526 99.314) (end 144.526 90.424) (angle 90) (layer Edge.Cuts) (width 0.1))
+  (gr_line (start 144.78 99.314) (end 144.526 99.314) (angle 90) (layer Edge.Cuts) (width 0.1))
+  (gr_line (start 153.416 99.314) (end 144.78 99.314) (angle 90) (layer Edge.Cuts) (width 0.1))
+  (gr_line (start 153.416 90.424) (end 153.416 99.314) (angle 90) (layer Edge.Cuts) (width 0.1))
+  (gr_line (start 144.526 90.424) (end 153.416 90.424) (angle 90) (layer Edge.Cuts) (width 0.1))
+  (segment (start 146.812 97.536) (end 146.304 97.028) (width 0.254) (layer F.Cu) (net 1))
+  (segment (start 146.304 97.028) (end 146.304 92.71) (width 0.254) (layer F.Cu) (net 1))
   (segment (start 147.828 97.536) (end 146.812 97.536) (width 0.254) (layer F.Cu) (net 1))
-  (segment (start 146.304 97.028) (end 146.304 92.71) (width 0.254) (layer F.Cu) (net 1))
-  (segment (start 146.812 97.536) (end 146.304 97.028) (width 0.254) (layer F.Cu) (net 1))
+  (segment (start 148.959 92.595) (end 148.844 92.71) (width 0.254) (layer F.Cu) (net 2))
+  (segment (start 151.638 92.595) (end 148.959 92.595) (width 0.254) (layer F.Cu) (net 2))
+  (segment (start 148.844 95.123) (end 149.098 95.377) (width 0.254) (layer F.Cu) (net 2))
+  (segment (start 149.098 95.377) (end 149.098 97.536) (width 0.254) (layer F.Cu) (net 2))
   (segment (start 148.844 92.71) (end 148.844 95.123) (width 0.254) (layer F.Cu) (net 2))
-  (segment (start 149.098 95.377) (end 149.098 97.536) (width 0.254) (layer F.Cu) (net 2))
-  (segment (start 148.844 95.123) (end 149.098 95.377) (width 0.254) (layer F.Cu) (net 2))
-  (segment (start 151.638 92.595) (end 148.959 92.595) (width 0.254) (layer F.Cu) (net 2))
-  (segment (start 148.959 92.595) (end 148.844 92.71) (width 0.254) (layer F.Cu) (net 2))
+  (segment (start 151.638 96.266) (end 150.368 97.536) (width 0.254) (layer F.Cu) (net 3))
   (segment (start 151.638 94.095) (end 151.638 96.266) (width 0.254) (layer F.Cu) (net 3))
-  (segment (start 151.638 96.266) (end 150.368 97.536) (width 0.254) (layer F.Cu) (net 3))
 )
